File: PCB/drone_fc/drone_fc.kicad_sch (KiCad schematic)
At the start: 45 parts, among them J1 USB_C_Receptacle_USB2.0_16P, J2 Conn_01x04_Socket, J3 Conn_01x08_Socket, SW1 PTS820J25M, U1 nRF52840, U2 USBLC6-2SC6, U3 ICM-20948, U4 MCP1703AT-3302E/DB, U5 LP5907MFX-1.8, U6 TCA9517A, X1 32MHz

Commit message: Back to the PCB now that I know the IMU works. I think most of the electrical connections are good (I'm still iffy on the nRF52840's VDD/VBUS stuff for hooking up a battery or USB), so I need to find components and run traces.
Parts:
- SW1: footprint SW2_PTS820J25MSMTRLFS_CNK -> footprints:SW2_PTS820J25MSMTRLFS_CNK
- U6: footprint (none) -> Package_SO:VSSOP-8_3x3mm_P0.65mm; symbol TCA9517A:TCA95177A -> Logic_LevelTranslator:TCA9517ADGK; Link (none) -> https://www.digikey.com/en/products/detail/texas-instrument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
- X1: Link (none) -> https://www.digikey.com/en/products/detail/ecs-inc/ECS-320-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
Connections:
- net SCL: now also J2.4 (Pin_4); no longer J2.3 (Pin_3)
- net SDA: now also J2.3 (Pin_3); no longer J2.4 (Pin_4)
- net at C13.1, U1.A23 (XC2): now also X1.3; no longer X1.2
Other:
- note added: "Ew. TODO: Fix this symbol"
- moved on the sheet: C24, C25

Commit message: Changed reset button, still need a header for SWD, and decided to move to a 4-layer board just to add some difficulty
Parts:
- added C26: 0u1, Capacitor_SMD:C_0402_1005Metric, symbol Device:C
- added D2: D_Schottky, Diode_SMD:Nexperia_CFP3_SOD-123W, symbol Device:D_Schottky
- C15: value 1u -> 100n
- SW1: value PTS820J25M -> PTS815SJM250SMTRLFS; footprint footprints:SW2_PTS820J25MSMTRLFS_CNK -> footprints:PTS815SJM250SMTRLFS; Link https://www.digikey.com/en/products/detail/c-k/PTS820J25MSM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 -> https://www.digikey.com/en/products/detail/c-k/PTS815SJM250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
Connections:
- net +15V: now also D2.2 (A); no longer C19.1, D1.1 (K), U4.1 (VI)
- net +1V8: now also C26.1
- net D+: now also U2.1 (I/O1); no longer U2.3 (I/O2)
- net D-: now also U2.3 (I/O2); no longer U2.1 (I/O1)
- net DR+: now also U2.6 (I/O1); no longer U2.4 (I/O2)
- net DR-: now also U2.4 (I/O2); no longer U2.6 (I/O1)
- net GND: now also SW1.4 (2), C26.2; no longer SW1.2
- new net: C19.1, D1.1 (K), D2.1 (K), U4.1 (VI)
Other:
- note added: "Fix this symbol too"
- moved on the sheet: C20

Commit message: Stepping back from PCB to ensure the schematic is actually done and to read up on better PCB design. Will likely start from scratch. Did add mounting holes since I completely forgot that earlier
Parts:
- removed D2: D_Schottky, Diode_SMD:Nexperia_CFP3_SOD-123W, symbol Device:D_Schottky
- added J4: Conn_ARM_SWD_TagConnect_TC2030, Connector:Tag-Connect_TC2030-IDC-FP_2x03_P1.27mm_Vertical, symbol Connector:Conn_ARM_SWD_TagConnect_TC2030
- D1: Link (none) -> https://www.digikey.com/en/products/detail/nexperia-usa-inc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
Connections:
- net +15V: now also C19.1, D1.1 (K), U4.1 (VI)
- net 3V3: now also J4.1 (VCC)
- net GND: now also J4.5 (GND)
- net NRESET: now also J4.3 (~{RESET})
- net SWDCLK: now also J4.4 (SWCLK)
- net SWDIO: now also J4.2 (SWDIO)
- net SWO: now reaches U1.AD22 (TRACEDATA0/P1.00)
- net SWO: now also J4.6 (SWO)
- no-connect marks 11 -> 12
Changed lines of the file:
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@@
 	)
 	(no_connect
+		(at 494.03 207.01)
+	)
+	(no_connect
 		(at 257.81 190.5)
 	)
@@
 	(wire
 		(pts
-			(xy 515.62 323.85) (xy 535.94 323.85)
+			(xy 499.11 311.15) (xy 519.43 311.15)
 		)
 		(stroke
@@
 	(wire
 		(pts
-			(xy 156.21 213.36) (xy 156.21 214.63)
+			(xy 156.21 213.36) (xy 156.21 223.52)
 		)
 		(stroke
@@
 	(wire
 		(pts
-			(xy 156.21 222.25) (xy 156.21 223.52)
-		)
-		(stroke
-			(width 0)
-			(type default)
-		)
-	)
-	(wire
-		(pts
 			(xy 361.95 166.37) (xy 355.6 166.37)
 		)
@@
 	(wire
 		(pts
-			(xy 515.62 326.39) (xy 535.94 326.39)
+			(xy 499.11 331.47) (xy 519.43 331.47)
 		)
 		(stroke
@@
 	(wire
 		(pts
-			(xy 90.17 312.42) (xy 90.17 314.96)
-		)
-		(stroke
-			(width 0)
-			(type default)
-		)
-	)
-	(wire
-		(pts
 			(xy 334.01 231.14) (xy 344.17 231.14)
 		)
@@
 	(wire
 		(pts
-			(xy 515.62 316.23) (xy 535.94 316.23)
+			(xy 316.23 246.38) (xy 316.23 254)
+		)
+		(stroke
+			(width 0)
+			(type default)
+		)
+	)
+	(wire
+		(pts
+			(xy 509.27 323.85) (xy 529.59 323.85)
 		)
 		(stroke
@@
 	(wire
 		(pts
+			(xy 316.23 254) (xy 323.85 254)
+		)
+		(stroke
+			(width 0)
+			(type default)
+		)
+	)
+	(wire
+		(pts
 			(xy 269.24 248.92) (xy 273.05 248.92)
 		)
@@
 	(wire
 		(pts
-			(xy 515.62 321.31) (xy 535.94 321.31)
+			(xy 509.27 316.23) (xy 529.59 316.23)
 		)
 		(stroke
@@
 	(wire
 		(pts
-			(xy 515.62 318.77) (xy 535.94 318.77)
+			(xy 509.27 321.31) (xy 529.59 321.31)
 		)
 		(stroke
@@
 	(wire
 		(pts
+			(xy 509.27 326.39) (xy 529.59 326.39)
+		)
+		(stroke
+			(width 0)
+			(type default)
+		)
+	)
+	(wire
+		(pts
 			(xy 97.79 367.03) (xy 97.79 364.49)
 		)
@@
 	)
 	(label "NRESET"
-		(at 535.94 321.31 180)
+		(at 529.59 316.23 180)
 		(effects
 			(font
@@
 	)
 	(label "GND"
-		(at 535.94 326.39 180)
+		(at 519.43 331.47 180)
 		(effects
 			(font
@@
 		)
 	)
+	(label "SWO"
+		(at 529.59 326.39 180)
+		(effects
+			(font
+				(size 1.27 1.27)
+			)
+			(justify right bottom)
+		)
+	)
 	(label "3V3"
 		(at 535.94 304.8 180)
@@
 	)
 	(label "SWDCLK"
-		(at 535.94 318.77 180)
+		(at 529.59 321.31 180)
 		(effects
 			(font
@@
 	)
 	(label "3V3"
-		(at 535.94 323.85 180)
+		(at 519.43 311.15 180)
 		(effects
 			(font
@@
 	)
 	(label "SWDIO"
-		(at 535.94 316.23 180)
+		(at 529.59 323.85 180)
+		(effects
+			(font
+				(size 1.27 1.27)
+			)
+			(justify right bottom)
+		)
+	)
+	(label "SWO"
+		(at 323.85 254 180)
 		(effects
 			(font
@@
 			)
 		)
+		(property "Link" "https://www.digikey.com/en/products/detail/nexperia-usa-inc/PMEG6020ER-115/2296182"
+			(at 168.91 218.44 0)
+			(effects
+				(font
+					(size 1.27 1.27)
+				)
+				(hide yes)
+			)
+		)
 		(pin "2"
 		)
@@
 	(symbol
 		(lib_id "power:PWR_FLAG")
-		(at 90.17 312.42 0)
+		(at 90.17 314.96 0)
 		(unit 1)
 		(exclude_from_sim no)
@@
 		(fields_autoplaced yes)
 		(property "Reference" "#FLG04"
-			(at 90.17 310.515 0)
+			(at 90.17 313.055 0)
 			(effects
 				(font
@@
 		)
 		(property "Value" "PWR_FLAG"
-			(at 90.17 307.34 0)
+			(at 90.17 309.88 0)
 			(effects
 				(font
@@
 		)
 		(property "Footprint" ""
-			(at 90.17 312.42 0)
+			(at 90.17 314.96 0)
 			(effects
 				(font
@@
 		)
 		(property "Datasheet" "~"
-			(at 90.17 312.42 0)
+			(at 90.17 314.96 0)
 			(effects
 				(font
@@
 		)
 		(property "Description" "Special symbol for telling ERC where power comes from"
-			(at 90.17 312.42 0)
+			(at 90.17 314.96 0)
 			(effects
 				(font
@@
 	)
 	(symbol
+		(lib_id "Connector:Conn_ARM_SWD_TagConnect_TC2030")
+		(at 501.65 321.31 0)
+		(unit 1)
+		(exclude_from_sim no)
+		(in_bom no)
+		(on_board yes)
+		(dnp no)
+		(fields_autoplaced yes)
+		(property "Reference" "J4"
+			(at 495.3 320.0399 0)
+			(effects
+				(font
+					(size 1.27 1.27)
+				)
+				(justify right)
+			)
+		)
+		(property "Value" "Conn_ARM_SWD_TagConnect_TC2030"
+			(at 495.3 322.5799 0)
+			(effects
+				(font
+					(size 1.27 1.27)
+				)
+				(justify right)
+				(hide yes)
+			)
+		)
+		(property "Footprint" "Connector:Tag-Connect_TC2030-IDC-FP_2x03_P1.27mm_Vertical"
+			(at 501.65 339.09 0)
+			(effects
+				(font
+					(size 1.27 1.27)
+				)
+				(hide yes)
+			)
+		)
+		(property "Datasheet" "https://www.tag-connect.com/wp-content/uploads/bsk-pdf-manager/TC2030-CTX_1.pdf"
+			(at 501.65 336.55 0)
+			(effects
+				(font
+					(size 1.27 1.27)
+				)
+				(hide yes)
+			)
+		)
+		(property "Description" "Tag-Connect ARM Cortex SWD JTAG connector, 6 pin"
+			(at 501.65 321.31 0)
+			(effects
+				(font
+					(size 1.27 1.27)
+				)
+				(hide yes)
+			)
+		)
+		(pin "3"
+		)
+		(pin "5"
+		)
+		(pin "4"
+		)
+		(pin "2"
+		)
+		(pin "6"
+		)
+		(pin "1"
+		)
+		(instances
+			(project ""
+				(path "/0506b644-0d93-4e3b-af7b-42a60683a977"
+					(reference "J4")
+					(unit 1)
+				)
+			)
+		)
+	)
+	(symbol
 		(lib_id "Device:C")
 		(at 351.79 154.94 90)
@@
 					(unit 1)
 				)
-			)
-		)
-	)
-	(symbol
-		(lib_id "Device:D_Schottky")
-		(at 156.21 218.44 90)
-		(unit 1)
-		(exclude_from_sim no)
-		(in_bom yes)
-		(on_board yes)
-		(dnp no)
-		(property "Reference" "D2"
-			(at 151.638 217.424 90)
-			(effects
-				(font
-					(size 1.27 1.27)
-				)
-				(justify right)
-			)
-		)
-		(property "Value" "D_Schottky"
-			(at 144.018 219.456 90)
-			(effects
-				(font
-					(size 1.27 1.27)
-				)
-				(justify right)
-			)
-		)
-		(property "Footprint" "Diode_SMD:Nexperia_CFP3_SOD-123W"
-			(at 156.21 218.44 0)
-			(effects
-				(font
-					(size 1.27 1.27)
-				)
-				(hide yes)
-			)
-		)
-		(property "Datasheet" "~"
-			(at 156.21 218.44 0)
-			(effects
-				(font
-					(size 1.27 1.27)
-				)
-				(hide yes)
-			)
-		)
-		(property "Description" "Schottky diode"
-			(at 156.21 218.44 0)
-			(effects
-				(font
-					(size 1.27 1.27)
-				)
-				(hide yes)
-			)
-		)
-		(pin "2"
-		)
-		(pin "1"
-		)
-		(instances
-			(project "drone_fc"
-				(path "/0506b644-0d93-4e3b-af7b-42a60683a977"
-					(reference "D2")
-					(unit 1)
-				)

Commit message: It's... done? I still have to create and route the VL53L4CX interrupt signal but otherwise I think this just needs some more grounding. I made sure that vias weren't on top of unrelated traces just in case JLCPCB doesn't support blind vias on their basic PCBs, but if they don't then I'm not sure what I'm going to do about the NRESET pin or the large die pad. I might have to contact them.
Parts:
- removed C24, C25: 1u, Capacitor_SMD:C_0603_1608Metric, symbol Device:C
- removed U6: TCA9517A, Package_SO:VSSOP-8_3x3mm_P0.65mm, symbol Logic_LevelTranslator:TCA9517ADGK
- added Q1: BSS138, Package_TO_SOT_SMD:SOT-323_SC-70, symbol Transistor_FET:BSS138
- added Q3: BSS138BKS, Package_TO_SOT_SMD:SOT-363_SC-70-6, symbol BSS_138_2:BSS_138
- added R7, R8: 4k7, Resistor_SMD:R_0402_1005Metric, symbol Device:R
- C11: renamed from C15; footprint Capacitor_SMD:C_0603_1608Metric -> Capacitor_SMD:C_0402_1005Metric
- C12: renamed from C7; footprint Capacitor_SMD:C_0603_1608Metric -> Capacitor_SMD:C_0402_1005Metric
- C4: renamed from C5; footprint Capacitor_SMD:C_0603_1608Metric -> Capacitor_SMD:C_0402_1005Metric
- C9: renamed from C6; footprint Capacitor_SMD:C_0603_1608Metric -> Capacitor_SMD:C_0402_1005Metric
- J2: renamed from J4; footprint Connector:Tag-Connect_TC2030-IDC-FP_2x03_P1.27mm_Vertical -> Connector:Tag-Connect_TC2030-IDC-NL_2x03_P1.27mm_Vertical
- R5: renamed from R3; footprint Resistor_SMD:R_0603_1608Metric -> Resistor_SMD:R_0402_1005Metric
- R6: renamed from R4; footprint Resistor_SMD:R_0603_1608Metric -> Resistor_SMD:R_0402_1005Metric
- U2: renamed from U4; value MCP1703AT-3302E/DB -> MCP1703AT-3302E/MB; footprint Package_TO_SOT_SMD:SOT-223-3_TabPin2 -> Package_TO_SOT_SMD:SOT-89-3; symbol Regulator_Linear:MCP1703Ax-330xxDB -> Regulator_Linear:MCP1703Ax-330xxMB; Link https://www.digikey.com/en/products/detail/microchip-technology/mcp1703at-3302e-db/3131473 -> https://www.digikey.com/en/products/detail/microchip-technology/MCP1703AT-3302E-MB/3131474
- renumbered C19 to C1, C14 to C10, C12 to C14, C16 to C15, C11 to C16, C10 to C17, C17 to C18, C18 to C19, C20 to C2, C3 to C21, C23 to C22, C26 to C24, C22 to C25, C21 to C26, C4 to C3, C8 to C5, C1 to C6, C2 to C7, C9 to C8, J2 to J3, J3 to J4, R5 to R3, R6 to R4, U2 to U1, U1 to U3, U5 to U4, U3 to U6
Connections:
- net VDD is gone; now on net 3V3: R3.1, R4.1
- net +1V8: now also Q1.1 (G), Q3.2 (G), Q3.5 (G), R8.1
- net 3V3: now also R7.1
- net IMU_INT_1_8: now also Q1.2 (S), R8.2
- net NRESET: now also SW1.1, U3.AC13 (P0.18/~{RESET})
- net SCL: now also Q3.3 (D)
- net SDA: now also Q3.6 (D)
- net VBAT: no longer U3.A10 (AIN5/P0.29)
- net SCL_1_8: now reaches U6.23 (SCL/SCLK)
- net SCL_1_8: now also R5.2, Q3.4 (S); no longer R6.2
- net SDA_1_8: now reaches U6.24 (SDA/SDI)
- net SDA_1_8: now also R6.2, Q3.1 (S); no longer R5.2
- net IMU_INT: now reaches U3.L1 (P0.06)
- net IMU_INT: now also Q1.3 (D), R7.2
- no-connect marks 12 -> 50
Other:
- note removed: "Ew. TODO: Fix this symbol"
- note removed: "Will need a MOSFET for this"
- moved on the sheet: BT1, C1, C10, C11, C12, C13, C14, C15, C16, C17, C18, C19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
